Commit message: Write ball chaser robot package

File: 2-ROS Essentials/catkin_ws/src/my_robot/urdf/my_robot.xacro (robot description, xacro)
@@ -1,4 +1,5 @@
 <?xml version='1.0'?>
 <robot name="my_robot" xmlns:xacro="http://www.ros.org/wiki/xacro">
+  <xacro:include filename="$(find my_robot)/urdf/my_robot.gazebo" />
   <link name="robot_footprint"></link>
   <joint name="robot_footprint_joint" type="fixed">
@@ -107,8 +108,4 @@
           <box size="0.05 0.05 0.05"/>
         </geometry>
-        <material name="red">
-          <color rgba="1.0 0.0 0.0 1.0"/>
-          <texture filename=""/>
-        </material>
       </visual>
       <collision>
@@ -118,4 +115,7 @@
         </geometry>
       </collision>
+      <gazebo reference="camera">
+          <material>Gazebo/Green</material>
+      </gazebo>
     </link>
 <joint name="camera_joint" type="fixed">
